File: CNPEM - GPS Cape/GPS Cape.sch (KiCad schematic (older format))
At the start: 11 parts, among them J101 Adafruit_ultimate_GPS_breakout, U101 74LS123

Commit message: schematics and pcb finished
Parts:
- added unit 1 of Beagle101
- added C104, C105: 100n, Capacitors_SMD:C_0805_HandSoldering, symbol C
- added C106: 0.1u, Capacitors_SMD:C_0805_HandSoldering, symbol C
- added R103, R104: 10k, Resistors_SMD:R_0805_HandSoldering, symbol R
Connections:
- net GND: now also Beagle101.C44, Beagle101.B1, C104.2, C105.2, C106.1
- net +3V3 renamed VCC
- net VCC: now also C104.1, C105.1, R103.1, R104.1; no longer C102.2, J101.2 (En), U101.3 (Clr)
- new net: C102.2, R103.2, U101.3 (Clr)
- new net: C106.2, J101.2 (En), R104.2
- no-connect marks 44 -> 88
Other:
- note added: "Capacitor de Ruído Alargador de Pulso"
- note added: "Capacitor de Ruído GPS"

Commit message: LED and components revised
Parts:
- added D102: LED, LEDs:LED_0805, symbol LED
- added Q101: Q_NPN_BEC, TO_SOT_Packages_SMD:SOT-23_Handsoldering, symbol Q_NPN_BEC
- added R105: 10k, Resistors_SMD:R_0805_HandSoldering, symbol R
- added R106: 100, Resistors_SMD:R_0805_HandSoldering, symbol R
- C101: value 10n -> 1u
- R101: value 200K -> 1M
Connections:
- net GND: now also Q101.2 (E); no longer Beagle101.B1, Beagle101.C44
- net PPS_ENL: now also R105.2
- net +5V: now reaches Beagle101.C6
- net +5V: now also D102.2 (A)
- new net: Q101.1 (B), R105.1
- new net: D102.1 (K), R106.1
- new net: Q101.3 (C), R106.2
- no-connect marks 88 -> 89
Other:
- note added: "LED PPS"
Changed lines of the file:
@@
 P 5250 1250
 F 0 "R101" V 5350 1200 50  0000 C CNN
-F 1 "200K" V 5250 1250 50  0000 C CNN
+F 1 "1M" V 5250 1250 50  0000 C CNN
 F 2 "Resistors_SMD:R_0805_HandSoldering" V 5180 1250 50  0001 C CNN
 F 3 "" H 5250 1250 50  0000 C CNN
@@
 P 5750 1250
 F 0 "C101" V 5850 1350 50  0000 L CNN
-F 1 "10n" V 5850 1050 50  0000 L CNN
+F 1 "1u" V 5850 1050 50  0000 L CNN
 F 2 "Capacitors_SMD:C_0805_HandSoldering" H 5788 1100 50  0001 C CNN
 F 3 "" H 5750 1250 50  0000 C CNN
@@
 NoConn ~ 7700 1350
 NoConn ~ 7700 1250
-NoConn ~ 8200 1150
 NoConn ~ 7700 1150
 Text Label 3300 1950 0    60   ~ 0
@@
 NoConn ~ 7700 950
 NoConn ~ 7700 1050
-Wire Wire Line
-	4650 1250 5100 1250
-Wire Wire Line
-	5400 1250 5600 1250
-Wire Wire Line
-	5900 1250 6700 1250
-Wire Wire Line
-	5550 1400 5550 1250
-Connection ~ 5550 1250
-Wire Notes Line
-	4350 3150 6950 3150
-Wire Notes Line
-	6950 3150 6950 900
-Wire Notes Line
-	6950 900  4350 900
-Wire Wire Line
-	4950 1150 4950 1250
-Connection ~ 4950 1250
-Wire Wire Line
-	5950 1400 5950 1250
-Connection ~ 5950 1250
-Wire Wire Line
-	4500 1900 4500 1850
-Wire Wire Line
-	4500 1850 5000 1850
-Wire Notes Line
-	1450 900  1450 3150
-Wire Notes Line
-	1450 3150 4050 3150
-Wire Notes Line
-	1450 900  4050 900
-Wire Wire Line
-	4650 3000 6050 3000
-Connection ~ 5750 3000
-Wire Wire Line
-	6350 3000 6550 3000
-Wire Wire Line
-	6550 3000 6550 1250
-Connection ~ 6550 1250
-Wire Notes Line
-	4350 900  4350 3150
-Wire Wire Line
-	3300 2250 3800 2250
-Wire Wire Line
-	3800 2250 3800 2850
-Wire Wire Line
-	3750 2400 3300 2400
-Wire Wire Line
-	1800 2650 1800 2800
-Wire Wire Line
-	1800 2800 3800 2800
-Connection ~ 3800 2800
-Wire Wire Line
-	2350 2250 1800 2250
-Connection ~ 1800 2250
-Wire Wire Line
-	1800 1900 1800 1800
-Wire Wire Line
-	1800 1500 1800 1400
-Wire Wire Line
-	1800 2200 1800 2350
-Connection ~ 2100 1400
-Wire Notes Line
-	4050 900  4050 3150
-Wire Wire Line
-	3750 1250 3750 2400
-Wire Wire Line
-	1800 1400 3750 1400
-Connection ~ 3750 1400
-Wire Wire Line
-	8200 1450 8350 1450
-Wire Wire Line
-	8350 1600 8300 1600
-Wire Wire Line
-	8300 1600 8300 1450
-Connection ~ 8300 1450
-Wire Wire Line
-	9050 1050 9050 1100
-Wire Wire Line
-	8950 950  8950 900
 $Comp
 L BeagleBone Beagle101
@@
 	1    0    0    -1
 $EndComp
-Wire Wire Line
-	8200 950  8950 950
 $Comp
 L VCC #PWR07
@@
 NoConn ~ 9600 1100
 $Comp
-L GND #PWR08
-U 1 1 578D0AF0
-P 9200 1000
-F 0 "#PWR08" H 9200 750 50  0001 C CNN
-F 1 "GND" H 9200 850 50  0000 C CNN
-F 2 "" H 9200 1000 50  0000 C CNN
-F 3 "" H 9200 1000 50  0000 C CNN
-	1    9200 1000
-	1    0    0    -1
-$EndComp
-Wire Wire Line
-	9200 1000 9600 1000
-$Comp
-L GND #PWR09
-U 1 1 578D2178
-P 8750 3050
-F 0 "#PWR09" H 8750 2800 50  0001 C CNN
-F 1 "GND" H 8750 2900 50  0000 C CNN
-F 2 "" H 8750 3050 50  0000 C CNN
-F 3 "" H 8750 3050 50  0000 C CNN
-	1    8750 3050
-	-1   0    0    1
-$EndComp
-Wire Wire Line
-	8200 3050 8750 3050
-$Comp
 L R R103
 U 1 1 578CDE9B
@@
 	1    0    0    -1
 $EndComp
-Wire Wire Line
-	4650 1250 4650 2300
-Wire Wire Line
-	4650 2600 4650 3000
 $Comp
 L C C104
@@
 $EndComp
 $Comp
-L VCC #PWR010
+L VCC #PWR08
 U 1 1 578CED58
 P 1750 3600
-F 0 "#PWR010" H 1750 3450 50  0001 C CNN
+F 0 "#PWR08" H 1750 3450 50  0001 C CNN
 F 1 "VCC" H 1750 3750 50  0000 C CNN
 F 2 "" H 1750 3600 50  0000 C CNN
@@
 $EndComp
 $Comp
-L GND #PWR011
+L GND #PWR09
 U 1 1 578CED8D
 P 1750 4150
-F 0 "#PWR011" H 1750 3900 50  0001 C CNN
+F 0 "#PWR09" H 1750 3900 50  0001 C CNN
 F 1 "GND" H 1750 4000 50  0000 C CNN
 F 2 "" H 1750 4150 50  0000 C CNN
@@
 	1    0    0    -1
 $EndComp
-Wire Wire Line
-	1750 4150 1750 4000
-Wire Wire Line
-	1750 3700 1750 3600
-Wire Notes Line
-	1450 3350 2200 3350
-Wire Notes Line
-	2200 3350 2200 4550
-Wire Notes Line
-	2200 4550 1450 4550
-Wire Notes Line
-	1450 4550 1450 3350
 Text Notes 1500 4500 0    60   ~ 0
 Capacitor de Ruído Alargador de Pulso
 $Comp
-L VCC #PWR012
+L VCC #PWR010
 U 1 1 578D2E37
 P 4100 3550
-F 0 "#PWR012" H 4100 3400 50  0001 C CNN
+F 0 "#PWR010" H 4100 3400 50  0001 C CNN
 F 1 "VCC" H 4100 3700 50  0000 C CNN
 F 2 "" H 4100 3550 50  0000 C CNN
@@
 $EndComp
 $Comp
-L GND #PWR013
+L GND #PWR011
 U 1 1 578D2F07
 P 4100 4200
-F 0 "#PWR013" H 4100 3950 50  0001 C CNN
+F 0 "#PWR011" H 4100 3950 50  0001 C CNN
 F 1 "GND" H 4100 4050 50  0000 C CNN
 F 2 "" H 4100 4200 50  0000 C CNN
@@
 	1    0    0    -1
 $EndComp
-Wire Wire Line
-	4100 3550 4100 3700
-Wire Wire Line
-	4100 4200 4100 4000
-Wire Notes Line
-	3700 3250 3700 4550
-Wire Notes Line
-	3700 4550 4800 4550
-Wire Notes Line
-	4800 4550 4800 3250
-Wire Notes Line
-	4800 3250 3700 3250
 Text Notes 3750 4500 0    60   ~ 0
 Capacitor de Ruído GPS
-Wire Wire Line
-	8200 1050 9050 1050
 $Comp
 L R R104
@@
 	-1   0    0    1
 $EndComp
+NoConn ~ 9600 1000
+NoConn ~ 8200 3050
+$Comp
+L +5V #PWR012
+U 1 1 578F8DA9
+P 8800 1150
+F 0 "#PWR012" H 8800 1000 50  0001 C CNN
+F 1 "+5V" H 8800 1290 50  0000 C CNN
+F 2 "" H 8800 1150 50  0000 C CNN
+F 3 "" H 8800 1150 50  0000 C CNN
+	1    8800 1150
+	-1   0    0    1
+$EndComp
+$Comp
+L +5V #PWR013
+U 1 1 578F95AD
+P 6650 3450
+F 0 "#PWR013" H 6650 3300 50  0001 C CNN
+F 1 "+5V" H 6650 3590 50  0000 C CNN
+F 2 "" H 6650 3450 50  0000 C CNN
+F 3 "" H 6650 3450 50  0000 C CNN
+	1    6650 3450
+	1    0    0    -1
+$EndComp
+Text Label 5800 4900 2    60   ~ 0
+PPS_ENL
+$Comp
+L GND #PWR014
+U 1 1 578F9ED2
+P 6650 5200
+F 0 "#PWR014" H 6650 4950 50  0001 C CNN
+F 1 "GND" H 6650 5050 50  0000 C CNN
+F 2 "" H 6650 5200 50  0000 C CNN
+F 3 "" H 6650 5200 50  0000 C CNN
+	1    6650 5200
+	1    0    0    -1
+$EndComp
+$Comp
+L R R105
+U 1 1 578FA259
+P 6100 4900
+F 0 "R105" V 6200 4900 50  0000 C CNN
+F 1 "10k" V 6100 4900 50  0000 C CNN
+F 2 "Resistors_SMD:R_0805_HandSoldering" V 6030 4900 50  0001 C CNN
+F 3 "" H 6100 4900 50  0000 C CNN
+	1    6100 4900
+	0    1    1    0
+$EndComp
+Wire Wire Line
+	4650 1250 5100 1250
+Wire Wire Line
+	5400 1250 5600 1250
+Wire Wire Line
+	5900 1250 6700 1250
+Wire Wire Line
+	5550 1400 5550 1250
+Connection ~ 5550 1250
+Wire Notes Line
+	4350 3150 6950 3150
+Wire Notes Line
+	6950 3150 6950 900
+Wire Notes Line
+	6950 900  4350 900
+Wire Wire Line
+	4950 1150 4950 1250
+Connection ~ 4950 1250
+Wire Wire Line
+	5950 1400 5950 1250
+Connection ~ 5950 1250
+Wire Wire Line
+	4500 1900 4500 1850
+Wire Wire Line
+	4500 1850 5000 1850
+Wire Notes Line
+	1450 900  1450 3150
+Wire Notes Line
+	1450 3150 4050 3150
+Wire Notes Line
+	1450 900  4050 900
+Wire Wire Line
+	4650 3000 6050 3000
+Connection ~ 5750 3000
+Wire Wire Line
+	6350 3000 6550 3000
+Wire Wire Line
+	6550 3000 6550 1250
+Connection ~ 6550 1250
+Wire Notes Line
+	4350 900  4350 3150
+Wire Wire Line
+	3300 2250 3800 2250
+Wire Wire Line
+	3800 2250 3800 2850
+Wire Wire Line
+	3750 2400 3300 2400
+Wire Wire Line
+	1800 2650 1800 2800
+Wire Wire Line
+	1800 2800 3800 2800
+Connection ~ 3800 2800
+Wire Wire Line
+	2350 2250 1800 2250
+Connection ~ 1800 2250
+Wire Wire Line
+	1800 1900 1800 1800
+Wire Wire Line
+	1800 1500 1800 1400
+Wire Wire Line
+	1800 2200 1800 2350
+Connection ~ 2100 1400
+Wire Notes Line
+	4050 900  4050 3150
+Wire Wire Line
+	3750 1250 3750 2400
+Wire Wire Line
+	1800 1400 3750 1400
+Connection ~ 3750 1400
+Wire Wire Line
+	8200 1450 8350 1450
+Wire Wire Line
+	8350 1600 8300 1600
+Wire Wire Line
+	8300 1600 8300 1450
+Connection ~ 8300 1450
+Wire Wire Line
+	9050 1050 9050 1100
+Wire Wire Line
+	8950 950  8950 900
+Wire Wire Line
+	8200 950  8950 950
+Wire Wire Line
+	4650 1250 4650 2300
+Wire Wire Line
+	4650 2600 4650 3000
+Wire Wire Line
+	1750 4150 1750 4000
+Wire Wire Line
+	1750 3700 1750 3600
+Wire Notes Line
+	1450 3350 2200 3350
+Wire Notes Line
+	2200 3350 2200 4550
+Wire Notes Line
+	2200 4550 1450 4550
+Wire Notes Line
+	1450 4550 1450 3350
+Wire Wire Line
+	4100 3550 4100 3700
+Wire Wire Line
+	4100 4200 4100 4000
+Wire Notes Line
+	3700 3250 3700 4550
+Wire Notes Line
+	3700 4550 4800 4550
+Wire Notes Line
+	4800 4550 4800 3250
+Wire Notes Line
+	4800 3250 3700 3250
+Wire Wire Line
+	8200 1050 9050 1050
 Wire Wire Line
 	2100 2700 2100 2800
@@
 Wire Wire Line
 	2100 2000 2100 2400
+Wire Wire Line
+	8800 1150 8200 1150
+Wire Notes Line
+	5350 3250 7550 3250
+Wire Notes Line
+	5350 5450 7550 5450
+Wire Notes Line
+	5350 3250 5350 5450
+Wire Wire Line
+	5800 4900 5950 4900
+Wire Notes Line
+	7550 5450 7550 3250
+$Comp
+L R R106
+U 1 1 578FB69A
+P 6650 4350
+F 0 "R106" V 6730 4350 50  0000 C CNN
+F 1 "100" V 6650 4350 50  0000 C CNN
+F 2 "Resistors_SMD:R_0805_HandSoldering" V 6580 4350 50  0001 C CNN
+F 3 "" H 6650 4350 50  0000 C CNN
+	1    6650 4350
+	1    0    0    -1
+$EndComp
+$Comp
+L LED D102
+U 1 1 578FB6EB
+P 6650 3900
+F 0 "D102" H 6650 4000 50  0000 C CNN
+F 1 "LED" H 6650 3800 50  0000 C CNN
+F 2 "LEDs:LED_0805" H 6650 3900 50  0001 C CNN
+F 3 "" H 6650 3900 50  0000 C CNN
+	1    6650 3900
+	0    -1   -1   0
+$EndComp
+Wire Wire Line
+	6650 3700 6650 3450
+Wire Wire Line
+	6650 4200 6650 4100
+Text Notes 5450 3400 0    60   ~ 0
+LED PPS
+$Comp
+L Q_NPN_BEC Q101
+U 1 1 578FE3E0
+P 6550 4900
+F 0 "Q101" H 6850 4950 50  0000 R CNN
+F 1 "Q_NPN_BEC" H 7150 4850 50  0000 R CNN
+F 2 "TO_SOT_Packages_SMD:SOT-23_Handsoldering" H 6750 5000 50  0001 C CNN
+F 3 "" H 6550 4900 50  0000 C CNN
+	1    6550 4900
+	1    0    0    -1
+$EndComp
+Wire Wire Line
+	6650 4700 6650 4500
+Wire Wire Line
+	6350 4900 6250 4900
+Wire Wire Line
+	6650 5200 6650 5100
 $EndSCHEMATC

Commit message: cape finished
Connections:
- net +5V: now also Beagle101.C8; no longer Beagle101.C6
Changed lines of the file:
@@
 NoConn ~ 8200 1550
 NoConn ~ 8200 1350
-NoConn ~ 8200 1250
 NoConn ~ 7700 1350
 NoConn ~ 7700 1250
@@
 L +5V #PWR012
 U 1 1 578F8DA9
-P 8800 1150
-F 0 "#PWR012" H 8800 1000 50  0001 C CNN
-F 1 "+5V" H 8800 1290 50  0000 C CNN
-F 2 "" H 8800 1150 50  0000 C CNN
-F 3 "" H 8800 1150 50  0000 C CNN
-	1    8800 1150
-	-1   0    0    1
+P 8800 1250
+F 0 "#PWR012" H 8800 1100 50  0001 C CNN
+F 1 "+5V" H 8800 1390 50  0000 C CNN
+F 2 "" H 8800 1250 50  0000 C CNN
+F 3 "" H 8800 1250 50  0000 C CNN
+	1    8800 1250
+	1    0    0    -1
 $EndComp
 $Comp
@@
 Wire Wire Line
 	2100 2000 2100 2400
-Wire Wire Line
-	8800 1150 8200 1150
 Wire Notes Line
 	5350 3250 7550 3250
@@
 Wire Wire Line
 	6650 5200 6650 5100
+NoConn ~ 8200 1150
+Wire Wire Line
+	8800 1250 8200 1250
 $EndSCHEMATC
