File: CNPEM - GPS Cape/gps_case_v2.kicad_pcb (KiCad board)
At the start: 2 copper layers, 87 x 54.6 mm, 21 parts, among them J101 Adafruit_ultimate_GPS_breakout, Q101 Q_NPN_BEC, U101 74LS123

Commit message: cape finished
Connections:
- Beagle101 pad C6: +5V -> Net-(Beagle101-PadC6)
- Beagle101 pad C8: Net-(Beagle101-PadC8) -> +5V
Routing:
- net +5V: track 15.1 -> 15.9 mm
